File: YOTSUBA_GNSS-Receiver/YOTSUBA_GNSS-receiver_Orion_ver.1.6.1.brd (EAGLE design)
At the start: 60.1 x 26 mm, 51 parts, among them IC2 NJM12877F33-TE1, J1 USB4500-03-0-A_REVA, J2 DF37B-10DP-0.4V_53_, U1 CP2102N-A01-GQFN28, U2 SF1186B-2, U3 MAX2670GTB+T

Commit message: C10 modified
Parts:
- C10: value 1u -> 0.1u
Changed lines of the file:
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@@
 <attribute name="NAME" x="36.325" y="24.65" size="1.27" layer="51" align="center"/>
 </element>
-<element name="C10" library="rcl" package="C1608" package3d_urn="urn:adsk.eagle:package:23621/2" value="1u" x="33.4" y="20.3" smashed="yes" rot="R90">
+<element name="C10" library="rcl" package="C1608" package3d_urn="urn:adsk.eagle:package:23621/2" value="0.1u" x="33.4" y="20.3" smashed="yes" rot="R90">
 <attribute name="NAME" x="33.465" y="23.74" size="1.016" layer="51" ratio="10" rot="R90" align="center"/>
 <attribute name="POPULARITY" value="3" x="32.7" y="-12.15" size="1.778" layer="27" rot="R90" display="off"/>
