File: YOTSUBA_GNSS-Receiver/YOTSUBA_GNSS-receiver_Orion_ver.1.6.1.sch (EAGLE design)
At the start: 51 parts, among them IC2 NJM12877F33-TE1, J1 USB4500-03-0-A_REVA, J2 DF37B-10DP-0.4V_53_, U1 CP2102N-A01-GQFN28, U2 SF1186B-2, U3 MAX2670GTB+T

Commit message: C10 modified
Parts:
- C10: value 1u -> 0.1u
Changed lines of the file:
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@@
 <part name="GND21" library="supply1" library_urn="urn:adsk.eagle:library:371" deviceset="GND" device=""/>
 <part name="IC2" library="SamacSys_Parts" library_urn="urn:adsk.eagle:library:38878568" deviceset="NJM12877F33-TE1" device="" package3d_urn="urn:adsk.eagle:package:38878576/2"/>
-<part name="C10" library="rcl" deviceset="C-EU" device="C1608" package3d_urn="urn:adsk.eagle:package:23621/2" value="1u"/>
+<part name="C10" library="rcl" deviceset="C-EU" device="C1608" package3d_urn="urn:adsk.eagle:package:23621/2" value="0.1u"/>
 <part name="GND22" library="supply1" library_urn="urn:adsk.eagle:library:371" deviceset="GND" device=""/>
 <part name="C11" library="rcl" deviceset="C-EU" device="C1608" package3d_urn="urn:adsk.eagle:package:23621/2" value="0.22u"/>
